File: Schematic/FTDI_Adapter/FTDI_Adapter.kicad_pcb (KiCad board)
At the start: 2 copper layers, 32.6 x 13.5 mm, 15 parts, among them J1 USB_B_Micro, J2 FFC6, U1 FT232RL

Commit message: File cleanup
Other:
- board text added: "."
Changed lines of the file:
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@@
     (effects (font (size 0.8 0.8) (thickness 0.1)) (justify left bottom))
+  )
+  (gr_text "." (at 88.42 35.53) (layer "F.SilkS")
+    (effects (font (size 1.5 1.5) (thickness 0.3) bold) (justify left bottom))
   )
   (gr_text "PWR" (at 72.6 45.3) (layer "F.SilkS")
